File: elec/l1/l1.kicad_sch (KiCad schematic)
At the start: 109 parts, among them IC2 SN74LVC2G04DBVTG4, IC3 SN74LVC2G04DBVTG4, SW1 SW_Push, U1 CD74HC4067M, U10 XT30PW-F, U2 CD74HC4067M, U4 STM32F103CBTx, U5 VNH5050A-E, U6 VNH5050A-E, U6 XT30PW-F, U7 VNH5050A-E, U7 XT30PW-F, U8 VNH5050A-E, U8 XT30PW-F, Y1 8Mhz

Commit message: activation circuit, motor drivers removed from l1
Parts:
- removed IC2, IC3: SN74LVC2G04DBVTG4, SOT95P280X145-6N, symbol SN74LVC2G04DBVTG4:SN74LVC2G04DBVTG4
- removed U10, U6, U7, U8: XT30PW-F, XT30PW-F, symbol XT30PW-F:XT30PW-F
- removed U5, U6, U7, U8: VNH5050A-E, SOP50P1030X247-39N, symbol VNH5050A-E:VNH5050A-E
- added C11: C, symbol Device:C
- added D27: 1N5401, Diode_THT:D_DO-201AD_P15.24mm_Horizontal, symbol Diode:1N5401
- added Q1: STP75NF75, TO255P1040X460X2890-3, symbol STP75NF75:STP75NF75
- added R44: 20, symbol Device:R
- added U1: XT30PW-F, XT30PW-F, symbol XT30PW-F:XT30PW-F
- added U2: LTV-817S, Package_DIP:SMDIP-4_W9.53mm, symbol Isolator:LTV-817S
- 22p1: footprint (none) -> footprints:cap0603
- C1: renamed from C6; footprint (none) -> footprints:cap0603
- C2: renamed from C7; footprint (none) -> footprints:cap0603
- C3: renamed from C8; footprint (none) -> footprints:cap0603
- C4: renamed from C9; footprint (none) -> footprints:cap0603
- C5: renamed from C10; footprint (none) -> footprints:cap0603
- C7: renamed from C1; footprint (none) -> footprints:cap0603
- C8: renamed from C2; footprint (none) -> footprints:cap0603
- C?: footprint footprints:EIA-7343-D -> footprints:cap0603
- Crystal1: renamed from Y1; footprint (none) -> Crystal:Crystal_SMD_Abracon_ABM8G-4Pin_3.2x2.5mm
- D1, D12, D13, D14, D15, D16, D17, D18, D19, D2, D20, D21, D22, D23, D24, D3, D4, D5, D6, D7, D8: footprint (none) -> LED_SMD:LED_0603_1608Metric_Pad1.05x0.95mm_HandSolder
- D10: renamed from D9; footprint (none) -> LED_SMD:LED_0603_1608Metric_Pad1.05x0.95mm_HandSolder
- D11: renamed from D10; footprint (none) -> LED_SMD:LED_0603_1608Metric_Pad1.05x0.95mm_HandSolder
- D25: renamed from D26; footprint (none) -> LED_SMD:LED_0603_1608Metric_Pad1.05x0.95mm_HandSolder
- D9: renamed from D11; footprint (none) -> LED_SMD:LED_0603_1608Metric_Pad1.05x0.95mm_HandSolder
- H1, H10, H11, H12, H13, H14, H2, H3, H4, H5, H6, H7, H8, H9: footprint (none) -> MountingHole:MountingHole_3.2mm_M3_Pad
- L?: footprint footprints:0630 One Piece Inductor -> footprints:L_Sunlord_SWPA8040S
- R1: renamed from R39; footprint (none) -> Resistor_SMD:R_0603_1608Metric_Pad0.98x0.95mm_HandSolder
- R10: renamed from R21; footprint (none) -> Resistor_SMD:R_0603_1608Metric_Pad0.98x0.95mm_HandSolder
- R11: renamed from R22; footprint (none) -> Resistor_SMD:R_0603_1608Metric_Pad0.98x0.95mm_HandSolder
- R12: renamed from R4; footprint (none) -> Resistor_SMD:R_0603_1608Metric_Pad0.98x0.95mm_HandSolder
- R13: renamed from R23; footprint (none) -> Resistor_SMD:R_0603_1608Metric_Pad0.98x0.95mm_HandSolder
- R14: renamed from R5; footprint (none) -> Resistor_SMD:R_0603_1608Metric_Pad0.98x0.95mm_HandSolder
- R15: renamed from R24; footprint (none) -> Resistor_SMD:R_0603_1608Metric_Pad0.98x0.95mm_HandSolder
- R16: renamed from R6; footprint (none) -> Resistor_SMD:R_0603_1608Metric_Pad0.98x0.95mm_HandSolder
- R17: renamed from R25; footprint (none) -> Resistor_SMD:R_0603_1608Metric_Pad0.98x0.95mm_HandSolder
- R18: renamed from R7; footprint (none) -> Resistor_SMD:R_0603_1608Metric_Pad0.98x0.95mm_HandSolder
- R19: renamed from R26; footprint (none) -> Resistor_SMD:R_0603_1608Metric_Pad0.98x0.95mm_HandSolder
- R2: renamed from R40; footprint (none) -> Resistor_SMD:R_0603_1608Metric_Pad0.98x0.95mm_HandSolder
- R20: renamed from R8; footprint (none) -> Resistor_SMD:R_0603_1608Metric_Pad0.98x0.95mm_HandSolder
- R21: renamed from R27; footprint (none) -> Resistor_SMD:R_0603_1608Metric_Pad0.98x0.95mm_HandSolder
- R22: renamed from R9; footprint (none) -> Resistor_SMD:R_0603_1608Metric_Pad0.98x0.95mm_HandSolder
- R23: renamed from R28; footprint (none) -> Resistor_SMD:R_0603_1608Metric_Pad0.98x0.95mm_HandSolder
- R24: renamed from R10; footprint (none) -> Resistor_SMD:R_0603_1608Metric_Pad0.98x0.95mm_HandSolder
- R25: renamed from R29; footprint (none) -> Resistor_SMD:R_0603_1608Metric_Pad0.98x0.95mm_HandSolder
- R26: renamed from R11; footprint (none) -> Resistor_SMD:R_0603_1608Metric_Pad0.98x0.95mm_HandSolder
- R27: renamed from R30; footprint (none) -> Resistor_SMD:R_0603_1608Metric_Pad0.98x0.95mm_HandSolder
- R28: renamed from R12; footprint (none) -> Resistor_SMD:R_0603_1608Metric_Pad0.98x0.95mm_HandSolder
- R29: renamed from R31; footprint (none) -> Resistor_SMD:R_0603_1608Metric_Pad0.98x0.95mm_HandSolder
- R3: renamed from R41; footprint (none) -> Resistor_SMD:R_0603_1608Metric_Pad0.98x0.95mm_HandSolder
- R30: renamed from R13; footprint (none) -> Resistor_SMD:R_0603_1608Metric_Pad0.98x0.95mm_HandSolder
- R31: renamed from R32; footprint (none) -> Resistor_SMD:R_0603_1608Metric_Pad0.98x0.95mm_HandSolder
- R32: renamed from R14; footprint (none) -> Resistor_SMD:R_0603_1608Metric_Pad0.98x0.95mm_HandSolder
- R33: renamed from R18; footprint (none) -> Resistor_SMD:R_0603_1608Metric_Pad0.98x0.95mm_HandSolder
- R34: renamed from R33; footprint (none) -> Resistor_SMD:R_0603_1608Metric_Pad0.98x0.95mm_HandSolder
- R35: renamed from R34; footprint (none) -> Resistor_SMD:R_0603_1608Metric_Pad0.98x0.95mm_HandSolder
- R36: renamed from R15; footprint (none) -> Resistor_SMD:R_0603_1608Metric_Pad0.98x0.95mm_HandSolder
- R37: renamed from R35; footprint (none) -> Resistor_SMD:R_0603_1608Metric_Pad0.98x0.95mm_HandSolder
- R38: renamed from R16; footprint (none) -> Resistor_SMD:R_0603_1608Metric_Pad0.98x0.95mm_HandSolder
- R39: renamed from R36; footprint (none) -> Resistor_SMD:R_0603_1608Metric_Pad0.98x0.95mm_HandSolder
- R4: renamed from R1; footprint (none) -> Resistor_SMD:R_0603_1608Metric_Pad0.98x0.95mm_HandSolder
- R5: renamed from R19; footprint (none) -> Resistor_SMD:R_0603_1608Metric_Pad0.98x0.95mm_HandSolder
- R6: renamed from R2; footprint (none) -> Resistor_SMD:R_0603_1608Metric_Pad0.98x0.95mm_HandSolder
- R7: renamed from R20; footprint (none) -> Resistor_SMD:R_0603_1608Metric_Pad0.98x0.95mm_HandSolder
- R8: renamed from R3; footprint (none) -> Resistor_SMD:R_0603_1608Metric_Pad0.98x0.95mm_HandSolder
- R9: renamed from R17; footprint (none) -> Resistor_SMD:R_0603_1608Metric_Pad0.98x0.95mm_HandSolder
- SW1: footprint (none) -> Button_Switch_SMD:SW_Push_1P1T-MP_NO_Horizontal_Alps_SKRTLAE010
- renumbered U1 to U11, U2 to U12, U4 to U9
Connections:
- net +12V: now also D27.1 (K), U1.P1 (-)
- net +3V3: now also U2.4
- net GND: now also C11.2, Q1.3, U2.2
- new net: Q1.1, U2.3
- new net: D27.2 (A), Q1.2, R44.2, U1.P2 (+)
- new net: C11.1, R44.1
- new net Sol: U2.1
- no-connect marks 26 -> 18
Other:
- note added: "solenoid activation circuit"
- moved on the sheet: 22p1, C1, C2, C3, C4, C5, C7, C8, C?, Crystal1, D1, D10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

Commit message: Updated stuff
Parts:
- added J1: Conn_01x04, Connector:Joint-Tech_C5080WR-04P_1x04_P5.08mm_Vertical, symbol Connector_Generic:Conn_01x04
- Q1: footprint TO255P1040X460X2890-3 -> footprints:TO255P1040X460X2890-3
- R42: renamed from R44; footprint (none) -> Resistor_SMD:R_0603_1608Metric_Pad0.98x0.95mm_HandSolder
- U6: renamed from U1; footprint XT30PW-F -> XT30PW-F:AMASS_XT30PW-F
- renumbered C8 to C10, C1 to C4, C2 to C5, C3 to C6, C4 to C7, C5 to C8, C7 to C9, D11 to D10, D12 to D11, D13 to D12, D14 to D13, D15 to D14, D16 to D15, D17 to D16, D18 to D17, D19 to D18, D9 to D26, D10 to D9, R8 to R10, R9 to R11, R10 to R12, R11 to R13, R12 to R14, R13 to R15, R14 to R16, R15 to R17, R16 to R18, R17 to R19, R18 to R20, R19 to R21, R20 to R22, R21 to R23, R22 to R24, R23 to R25, R24 to R26, R25 to R27, R26 to R28, R27 to R29, R1 to R3, R28 to R30, R29 to R31, R30 to R32, R31 to R33, R32 to R34, R33 to R35, R34 to R36, R35 to R37, R36 to R38, R37 to R39, R2 to R4, R38 to R40, R39 to R41, R3 to R5, R4 to R6, R5 to R7, R6 to R8, R7 to R9, U9 to U2, U11 to U3, U12 to U4, U2 to U5
Connections:
- net +3V3: now also J1.1 (Pin_1)
- net GND: now also J1.4 (Pin_4)
- net M1: now reaches R13.1, U4.1 (COM)
- net M1_S0: now reaches U4.10 (S0)
- net M1_S1: now reaches U4.11 (S1)
- net M1_S3: now reaches U4.13 (S3)
- net M1_S2: now reaches U4.14 (S2)
- net M2: now reaches R11.1, U3.1 (COM)
- net M2_S0: now reaches U3.10 (S0)
- net M2_S1: now reaches U3.11 (S1)
- net M2_S3: now reaches U3.13 (S3)
- net M2_S2: now reaches U3.14 (S2)
- new net rx: J1.2 (Pin_2)
- new net tx: J1.3 (Pin_3)

Commit message: stuff
Parts:
- removed 22p1: C5, footprints:cap0603, symbol Device:C
- removed C10, C9: C, footprints:cap0603, symbol Device:C
- removed C11: C, symbol Device:C
- removed C4: 22p, footprints:cap0603, symbol Device:C
- removed C5, C6, C7, C8: 0.1u, footprints:cap0603, symbol Device:C
- removed C?: 220u, footprints:cap0603, symbol Device:C_Polarized
- removed C?: 10n, footprints:cap0603, symbol Device:C
- removed C?: 10u, footprints:cap0603, symbol Device:C
- removed Crystal1: 8Mhz, Crystal:Crystal_SMD_Abracon_ABM8G-4Pin_3.2x2.5mm, symbol Device:Crystal
- removed D1, D10, D11, D12, D13, D14, D15, D16, D17, D18, D2, D20, D21, D22, D23, D24, D25, D26, D3, D4, D5, D6, D7, D8, D9: LED, LED_SMD:LED_0603_1608Metric_Pad1.05x0.95mm_HandSolder, symbol Device:LED
- removed D27: 1N5401, Diode_THT:D_DO-201AD_P15.24mm_Horizontal, symbol Diode:1N5401
- removed D?: SS54, footprints:DIOM5025X220N, symbol Diode:B340
- removed H1, H10, H11, H12, H13, H14, H2, H3, H4, H5, H6, H7, H8, H9: MountingHole, MountingHole:MountingHole_3.2mm_M3_Pad, symbol Mechanical:MountingHole
- removed J1: Conn_01x04, Connector:Joint-Tech_C5080WR-04P_1x04_P5.08mm_Vertical, symbol Connector_Generic:Conn_01x04
- removed L?: 15uH, footprints:L_Sunlord_SWPA8040S, symbol Device:L_Iron
- removed Q1: STP75NF75, footprints:TO255P1040X460X2890-3, symbol STP75NF75:STP75NF75
- removed R10, R12, R14, R15, R16, R17, R18, R19, R20, R21, R22, R23, R24, R25, R26, R27, R28, R29, R30, R31, R32, R33, R34, R36, R38, R39, R40, R41, R6, R7, R8, R9: R_Photo, Resistor_SMD:R_0603_1608Metric_Pad0.98x0.95mm_HandSolder, symbol Device:R_Photo
- removed R11, R13, R35, R37, R5: R, Resistor_SMD:R_0603_1608Metric_Pad0.98x0.95mm_HandSolder, symbol Device:R
- removed R3: 10K, Resistor_SMD:R_0603_1608Metric_Pad0.98x0.95mm_HandSolder, symbol Device:R
- removed R4: 1K, Resistor_SMD:R_0603_1608Metric_Pad0.98x0.95mm_HandSolder, symbol Device:R
- removed R42: 20, Resistor_SMD:R_0603_1608Metric_Pad0.98x0.95mm_HandSolder, symbol Device:R
- removed R?: 5K9, footprints:res0603, symbol Device:R
- removed R?: 10K, footprints:res0603, symbol Device:R
- removed SW1: SW_Push, Button_Switch_SMD:SW_Push_1P1T-MP_NO_Horizontal_Alps_SKRTLAE010, symbol Switch:SW_Push
- removed U2: STM32F103CBTx, Package_QFP:LQFP-48_7x7mm_P0.5mm, symbol MCU_ST_STM32F1:STM32F103CBTx
- removed U3, U4: CD74HC4067M, Package_SO:SOIC-24W_7.5x15.4mm_P1.27mm, symbol 74xx:CD74HC4067M
- removed U5: LTV-817S, Package_DIP:SMDIP-4_W9.53mm, symbol Isolator:LTV-817S
- removed U6: XT30PW-F, XT30PW-F:AMASS_XT30PW-F, symbol XT30PW-F:XT30PW-F
- removed U?: TPS5430DDA, footprints:TI_SO-PowerPAD-8_ThermalVias, symbol Regulator_Switching:TPS5430DDA
- added C?: 0u1, Library:cap0603, symbol Device:C
- added C?: 0.1u, Library:cap0603, symbol vincent:C
- added C?: 220u, Library:EIA-7343-D, symbol Device:C_Polarized
- added C?: 10n, Library:cap0603, symbol Device:C
- added C?: 10u, Library:cap0603, symbol Device:C
- added D? (x15): LED, Library:LED-3528, symbol Device:LED
- added D?: SS54, Library:SMA (DO-214AC), symbol Diode:B340
- added J2: Conn_01x08, Connector_JST:JST_EH_B8B-EH-A_1x08_P2.50mm_Vertical, symbol Connector_Generic:Conn_01x08
- added J?: Conn_01x02, Library:AMASS_XT30-F, symbol Connector_Generic:Conn_01x02
- added KM? (x3), MTH? (x11): MountingHole_Pad, MountingHole:MountingHole_3.2mm_M3_Pad_Via, symbol Mechanical:MountingHole_Pad
- added L?: 15uH, Library:0630 One Piece Inductor, symbol Device:L_Iron
- added R? (x15): R_Photo, Library:ALS-PT19, symbol Device:R_Photo
- added R?: 10K, Library:res0603, symbol Device:R
- added R?: 10K, Library:res0603, symbol vincent:R
- added R?: 5K9, Library:res0603, symbol Device:R
- added R?: 3K24, Library:cap0603, symbol vincent:R
- added U?: CD74HC4067SM, Package_SO:SSOP-24_5.3x8.2mm_P0.65mm, symbol 74xx:CD74HC4067SM
- added U?: TPS5430DDA, Library:TI_SO-PowerPAD-8, symbol Regulator_Switching:TPS5430DDA
Connections:
- net +12V: now also J?.1 (Pin_1)
- net +3V3: now also C?.1, C?.1, C?.2, D?.2 (A), D?.2 (A), D?.2 (A), D?.2 (A), D?.2 (A), D?.2 (A), D?.2 (A), D?.2 (A), D?.2 (A), D?.2 (A), D?.2 (A), D?.2 (A), D?.2 (A), D?.2 (A), D?.2 (A), L?.2, R?.1, R?.1, R?.1, R?.1, R?.1, R?.1, R?.1, R?.1, R?.1, R?.1, R?.1, R?.1, R?.1, R?.1, R?.1, R?.1, U?.24 (VCC)
- net GND: now also C?.1, C?.2, C?.2, C?.2, D?.1 (K), D?.1 (K), D?.1 (K), D?.1 (K), D?.1 (K), D?.1 (K), D?.1 (K), D?.1 (K), D?.1 (K), D?.1 (K), D?.1 (K), D?.1 (K), D?.1 (K), D?.1 (K), D?.1 (K), D?.2 (A), J2.7 (Pin_7), J2.8 (Pin_8), J?.2 (Pin_2), R?.1, R?.1, R?.2, U?.12 (GND), U?.6 (GND), U?.9 (GNDPAD)
- net M1: now also J2.6 (Pin_6), R?.2, U?.1 (COM)
- net M1_S0: now also J2.2 (Pin_2), U?.10 (S0)
- net M1_S1: now also J2.3 (Pin_3), U?.11 (S1)
- net M1_S2: now also J2.4 (Pin_4), U?.14 (S2)
- net M1_S3: now also J2.5 (Pin_5), U?.13 (S3)
- new net: R?.2, U?.17 (I14)
- new net: R?.1, R?.2, U?.4 (VSENSE)
- new net: R?.2, U?.9 (I0)
- new net: C?.2, D?.1 (K), L?.1, U?.8 (PH)
- new net: R?.2, U?.15 (~{E})
- new net: R?.2, U?.18 (I13)
- new net: R?.2, U?.19 (I12)
- new net: R?.2, U?.2 (I7)
- new net: R?.2, U?.20 (I11)
- new net: R?.2, U?.21 (I10)
- new net: R?.2, U?.22 (I9)
- new net: R?.2, U?.23 (I8)
- new net: R?.2, U?.3 (I6)
- new net: R?.2, U?.4 (I5)
- new net: R?.2, U?.5 (I4)
- new net: R?.2, U?.6 (I3)
- new net: R?.2, U?.7 (I2)
- new net: R?.2, U?.8 (I1)
- new net: C?.1, U?.1 (BOOT)
- new net +5V: C?.1, J2.1 (Pin_1), U?.7 (VIN)
- no-connect marks 18 -> 1
Other:
- note added: "3V3 Buck"
- note added: "Connection"
- note added: "LED"
- note added: "MTH"
- note added: "MUX"
- note removed: "solenoid activation circuit"

Commit message: ass
Changed lines of the file:
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@@
     (fill (type none))
   )
-  (rectangle (start 34.29 107.315) (end 140.97 188.595)
+  (rectangle (start 34.29 107.315) (end 140.97 159.385)
     (stroke (width 0) (type default))
     (fill (type none))
@@
       (project "l1"
         (path "/83813a76-0730-4df2-a3a5-0ea20d9ce8b3"
-          (reference "R33") (unit 1)
-        )
-      )
+          (reference "R1") (unit 1)
+        )
+      )
