File: elec/l1/l1.kicad_pcb (KiCad board)
At the start: 2 copper layers, 108 parts, among them IC1 SN74LVC2G04DBVTG4, IC2 SN74LVC2G04DBVTG4, SW1 SW_Push, U1 XT30PW-F, U11 CD74HC4067M, U12 CD74HC4067M, U2 XT30PW-F, U3 XT30PW-F, U4 XT30PW-F, U5 VNH5050A-E, U6 VNH5050A-E, U7 VNH5050A-E, U8 VNH5050A-E, U9 STM32F103CBTx

Commit message: Updated stuff
Parts:
- added D27: 1N5401, Diode_THT:D_DO-201AD_P15.24mm_Horizontal, F.Cu at (128.4, -13.2)
- added J1: Conn_01x04, Connector:Joint-Tech_C5080WR-04P_1x04_P5.08mm_Vertical, F.Cu at (133.4, -41.4)
- added Q1: STP75NF75, footprints:TO255P1040X460X2890-3, F.Cu at (159.5, -15.7)
- added R42: 20, Resistor_SMD:R_0603_1608Metric_Pad0.98x0.95mm_HandSolder, F.Cu at (158.2, -11.6)
- added U5: LTV-817S, Package_DIP:SMDIP-4_W9.53mm, F.Cu at (162.7, -22.4)
- added U6: XT30PW-F, XT30PW-F:AMASS_XT30PW-F, F.Cu at (163.5, -34.0)
- renumbered C6 to C1, C8 to C10, C9 to C2, C10 to C3, C1 to C4, C2 to C5, C3 to C6, C4 to C7, C5 to C8, C7 to C9, D11 to D10, D12 to D11, D13 to D12, D14 to D13, D15 to D14, D16 to D15, D17 to D16, D18 to D17, D19 to D18, D26 to D19, D9 to D26, D10 to D9, R40 to R1, R8 to R10, R9 to R11, R10 to R12, R11 to R13, R12 to R14, R13 to R15, R14 to R16, R15 to R17, R16 to R18, R17 to R19, R41 to R2, R18 to R20, R19 to R21, R20 to R22, R21 to R23, R22 to R24, R23 to R25, R24 to R26, R25 to R27, R26 to R28, R27 to R29, R1 to R3, R28 to R30, R29 to R31, R30 to R32, R31 to R33, R32 to R34, R33 to R35, R34 to R36, R35 to R37, R36 to R38, R37 to R39, R2 to R4, R38 to R40, R39 to R41, R3 to R5, R4 to R6, R5 to R7, R6 to R8, R7 to R9, U9 to U2, U11 to U3, U12 to U4
Connections:
- net Net-(U11-COM) renamed /M2
- net Net-(U12-COM) renamed /M1
- U3 pad 10: unconnected-(U11-S0-Pad10) -> /M2_S0
- U3 pad 11: unconnected-(U11-S1-Pad11) -> /M2_S1
- U3 pad 13: unconnected-(U11-S3-Pad13) -> /M2_S3
- U3 pad 14: unconnected-(U11-S2-Pad14) -> /M2_S2
- U4 pad 10: unconnected-(U12-S0-Pad10) -> /M1_S0
- U4 pad 11: unconnected-(U12-S1-Pad11) -> /M1_S1
- U4 pad 13: unconnected-(U12-S3-Pad13) -> /M1_S3
- U4 pad 14: unconnected-(U12-S2-Pad14) -> /M1_S2

Commit message: stuff
Parts:
- removed 22p1: C5, footprints:cap0603
- removed C10, C9: C, footprints:cap0603
- removed C6, C7, C8: 0.1u, footprints:cap0603
- removed Crystal1: 8Mhz, Crystal:Crystal_SMD_Abracon_ABM8G-4Pin_3.2x2.5mm
- removed D17, D18, D20, D21, D22, D23, D24, D25, D26: LED, LED_SMD:LED_0603_1608Metric_Pad1.05x0.95mm_HandSolder
- removed D19: SS54, footprints:DIOM5025X220N
- removed D27: 1N5401, Diode_THT:D_DO-201AD_P15.24mm_Horizontal
- removed H1, H10, H11, H12, H13, H14, H2, H3, H4, H5, H6, H7, H8, H9: MountingHole, MountingHole:MountingHole_3.2mm_M3_Pad
- removed IC1, IC2: SN74LVC2G04DBVTG4, footprints:SOT95P280X145-6N
- removed Q1: STP75NF75, footprints:TO255P1040X460X2890-3
- removed R1: 5K9, footprints:res0603
- removed R20, R21, R22, R23, R24, R25, R26, R27, R28, R29, R30, R31, R32, R34, R36, R38, R39, R40, R41: R_Photo, Resistor_SMD:R_0603_1608Metric_Pad0.98x0.95mm_HandSolder
- removed R35, R37: R, Resistor_SMD:R_0603_1608Metric_Pad0.98x0.95mm_HandSolder
- removed R42: 20, Resistor_SMD:R_0603_1608Metric_Pad0.98x0.95mm_HandSolder
- removed SW1: SW_Push, Button_Switch_SMD:SW_Push_1P1T-MP_NO_Horizontal_Alps_SKRTLAE010
- removed the U2 at (58.5, -14.4)
- removed the U2 at (99.2, -57.5)
- removed U3, U4: CD74HC4067M, Package_SO:SOIC-24W_7.5x15.4mm_P1.27mm
- removed U3, U4: XT30PW-F, footprints:AMASS_XT30-F
- removed U5, U6, U7, U8: VNH5050A-E, footprints:SOP50P1030X247-39N
- removed U5: LTV-817S, Package_DIP:SMDIP-4_W9.53mm
- removed U6: XT30PW-F, XT30PW-F:AMASS_XT30PW-F
- added J2: Conn_01x08, Connector_JST:JST_EH_B8B-EH-A_1x08_P2.50mm_Vertical, F.Cu at (-11.3, 84.0)
- added MTH1: MountingHole_Pad, MountingHole:MountingHole_3.2mm_M3_Pad_Via, F.Cu at (78.3, 95.4)
- added MTH10: MountingHole_Pad, MountingHole:MountingHole_3.2mm_M3_Pad_Via, F.Cu at (140.5, 157.6)
- added MTH11: MountingHole_Pad, MountingHole:MountingHole_3.2mm_M3_Pad_Via, F.Cu at (78.3, 135.7)
- added MTH12: MountingHole_Pad, MountingHole:MountingHole_3.2mm_M3_Pad_Via, F.Cu at (199.2, 90.3)
- added MTH13: MountingHole_Pad, MountingHole:MountingHole_3.2mm_M3_Pad_Via, F.Cu at (199.2, 140.7)
- added MTH14: MountingHole_Pad, MountingHole:MountingHole_3.2mm_M3_Pad_Via, F.Cu at (100.2, 157.6)
- added MTH2: MountingHole_Pad, MountingHole:MountingHole_3.2mm_M3_Pad_Via, F.Cu at (162.4, 135.7)
- added MTH3: MountingHole_Pad, MountingHole:MountingHole_3.2mm_M3_Pad_Via, F.Cu at (93.2, 36.7)
- added MTH4: MountingHole_Pad, MountingHole:MountingHole_3.2mm_M3_Pad_Via, F.Cu at (100.2, 73.4)
- added MTH5: MountingHole_Pad, MountingHole:MountingHole_3.2mm_M3_Pad_Via, F.Cu at (147.6, 36.7)
- added MTH6: MountingHole_Pad, MountingHole:MountingHole_3.2mm_M3_Pad_Via, F.Cu at (41.6, 90.3)
- added MTH7: MountingHole_Pad, MountingHole:MountingHole_3.2mm_M3_Pad_Via, F.Cu at (162.4, 95.4)
- added MTH8: MountingHole_Pad, MountingHole:MountingHole_3.2mm_M3_Pad_Via, F.Cu at (41.6, 140.7)
- added MTH9: MountingHole_Pad, MountingHole:MountingHole_3.2mm_M3_Pad_Via, F.Cu at (140.5, 73.4)
- added U2: TPS5430DDA, Library:TI_SO-PowerPAD-8, F.Cu at (84.8, 114.7)
- C1: value 10u -> 0.1u; footprint footprints:cap0603 -> Library:cap0603
- C2: footprint footprints:cap0603 -> Library:cap0603
- C3: footprint footprints:cap0603 -> Library:EIA-7343-D
- C4: value 22p -> 0u1; footprint footprints:cap0603 -> Library:cap0603
- C5: value 0.1u -> 10u; footprint footprints:cap0603 -> Library:cap0603
- D1, D10, D11, D12, D13, D14, D15, D2, D3, D4, D5, D6, D7, D8, D9: footprint LED_SMD:LED_0603_1608Metric_Pad1.05x0.95mm_HandSolder -> Library:LED-3528; moved to B.Cu
- D16: value LED -> SS54; footprint LED_SMD:LED_0603_1608Metric_Pad1.05x0.95mm_HandSolder -> Library:SMA (DO-214AC)
- J1: value Conn_01x04 -> Conn_01x02; footprint Connector:Joint-Tech_C5080WR-04P_1x04_P5.08mm_Vertical -> Library:AMASS_XT30-F
- L1: footprint footprints:L_Sunlord_SWPA8040S -> Library:0630 One Piece Inductor
- R10, R12, R14, R15, R6, R7, R8, R9: footprint Resistor_SMD:R_0603_1608Metric_Pad0.98x0.95mm_HandSolder -> Library:ALS-PT19; moved to B.Cu
- R11, R13, R5: value R -> R_Photo; footprint Resistor_SMD:R_0603_1608Metric_Pad0.98x0.95mm_HandSolder -> Library:ALS-PT19; moved to B.Cu
- R16: value R_Photo -> 3K24; footprint Resistor_SMD:R_0603_1608Metric_Pad0.98x0.95mm_HandSolder -> Library:cap0603
- R17, R18: value R_Photo -> 10K; footprint Resistor_SMD:R_0603_1608Metric_Pad0.98x0.95mm_HandSolder -> Library:res0603
- R19: value R_Photo -> 5K9; footprint Resistor_SMD:R_0603_1608Metric_Pad0.98x0.95mm_HandSolder -> Library:res0603
- R2: value 10K -> R_Photo; footprint footprints:res0603 -> Library:ALS-PT19; moved to B.Cu
- R3: value 10K -> R_Photo; footprint Resistor_SMD:R_0603_1608Metric_Pad0.98x0.95mm_HandSolder -> Library:ALS-PT19; moved to B.Cu
- R33: footprint Resistor_SMD:R_0603_1608Metric_Pad0.98x0.95mm_HandSolder -> Library:ALS-PT19
- R4: value 1K -> R_Photo; footprint Resistor_SMD:R_0603_1608Metric_Pad0.98x0.95mm_HandSolder -> Library:ALS-PT19; moved to B.Cu
- U1: value XT30PW-F -> CD74HC4067SM; footprint footprints:AMASS_XT30-F -> Package_SO:SSOP-24_5.3x8.2mm_P0.65mm
- moved R4 234.0 mm to (108.4, 169.4), turned to 72 degrees
- moved R5 233.1 mm to (131.3, 169.6), turned to 96 degrees
- moved R3 227.6 mm to (87.5, 159.9), turned to 48 degrees
- moved R6 225.1 mm to (152.4, 160.4), turned to 120 degrees
- moved R17 223.0 mm to (-15.8, 127.7)
- moved R16 222.7 mm to (-15.8, 124.8)
- moved R33 221.1 mm to (-22.9, 103.3)
- moved R7 210.2 mm to (167.9, 143.5), turned to 144 degrees
- moved D2 204.5 mm to (142.4, 166.1), turned to -66 degrees
- moved D1 204.4 mm to (119.9, 170.7), turned to -90 degrees
- moved D3 197.7 mm to (161.0, 152.8), turned to -42 degrees
- moved J1 194.2 mm to (-9.01, 90.6)
- moved D15 191.4 mm to (97.5, 165.7), turned to -114 degrees
- moved R8 189.8 mm to (175.2, 121.8), turned to 168 degrees
- moved U1 184.6 mm to (2.12, 92.3)
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Connections:
- C1 pad 1: +12V -> GND
- C1 pad 2: GND -> +3V3
- C2 pad 2: Net-(D19-K) -> Net-(D16-K)
- C4 pad 1: GND -> +3V3
- C4 pad 2: Net-(U2-PD0) -> GND
- C5 pad 1: +3V3 -> +5V
- D16 pad 1: GND -> Net-(D16-K)
- D16 pad 2: +3V3 -> GND
- J1 pad 1: +3V3 -> +12V
- J1 pad 2: /rx -> GND
- L1 pad 1: Net-(D19-K) -> Net-(D16-K)
- R10 pad 2: Net-(U3-I2) -> Net-(U1-I9)
- R11 pad 1: /M2 -> +3V3
- R11 pad 2: GND -> Net-(U1-I10)
- R12 pad 2: Net-(U4-I2) -> Net-(U1-I11)
- R13 pad 1: /M1 -> +3V3
- R13 pad 2: GND -> Net-(U1-I12)
- R14 pad 2: Net-(U3-I3) -> Net-(U1-I13)
- R15 pad 2: Net-(U4-I3) -> Net-(U1-I14)
- R16 pad 1: +3V3 -> GND
- R16 pad 2: Net-(U3-I4) -> /M1
- R17 pad 1: +3V3 -> GND
- R17 pad 2: Net-(U4-I4) -> Net-(U1-~{E})
- R18 pad 2: Net-(U3-I5) -> Net-(U2-VSENSE)
- R19 pad 1: +3V3 -> Net-(U2-VSENSE)
- R19 pad 2: Net-(U4-I5) -> GND
- R2 pad 2: Net-(U1-VSENSE) -> Net-(U1-I1)
- R3 pad 2: Net-(R3-Pad2) -> Net-(U1-I2)
- R33 pad 2: Net-(U4-I12) -> Net-(U1-I0)
- R4 pad 1: Net-(R4-Pad1) -> +3V3
- R4 pad 2: GND -> Net-(U1-I3)
- R5 pad 1: GND -> +3V3
- R5 pad 2: /BOOT -> Net-(U1-I4)
- R6 pad 2: Net-(U3-I0) -> Net-(U1-I5)
- R7 pad 2: Net-(U4-I0) -> Net-(U1-I6)
- R8 pad 2: Net-(U3-I1) -> Net-(U1-I7)
- R9 pad 2: Net-(U4-I1) -> Net-(U1-I8)
- U1 pad 1: (no net) -> /M1
- U1 pad 2: (no net) -> Net-(U1-I7)
Routing:
- net Net-(U2-VSENSE): track 0.00 -> 7.38 mm
- net +3V3: track 0.00 -> 3.81 mm
- net (no net): vias 0 -> 1
- added copper zone on F.Cu, net +3V3
- added copper zone on F.Cu, net +5V
- added copper zone on B.Cu, net GND
- added copper zone on F.Cu, net GND
- added copper zone on F.Cu, net Net-(D16-K)
- added copper zone on F.Cu, net Net-(U2-BOOT)
Other:
- board outline added: 176 x 170.3 mm

Commit message: ass
Parts:
- removed R33: R_Photo, Library:ALS-PT19
- added R1: R_Photo, Library:ALS-PT19, B.Cu at (72.2, 143.3)
- moved J2 123.3 mm to (111.2, 97.6), turned to 90 degrees
- moved C1 119.6 mm to (102.3, 93.7)
- moved R16 119.6 mm to (102.3, 105.3)
- moved R17 119.6 mm to (102.3, 108.2)
- moved U1 119.6 mm to (120.2, 72.8)
- moved J1 95.8 mm to (85.6, 105.3)
- moved R4 23.5 mm to (131.9, 169.9), turned to -78 degrees
- moved R7 23.5 mm to (175.7, 121.3), turned to -6 degrees
- moved R14 23.5 mm to (67.5, 98.3), turned to 162 degrees
- moved R9 23.5 mm to (161.7, 78.3), turned to 42 degrees
- moved R10 23.5 mm to (143.0, 64.7), turned to 66 degrees
- moved R12 23.5 mm to (97.7, 64.7), turned to 114 degrees
- moved R5 23.5 mm to (153.1, 160.5), turned to -54 degrees
- moved R8 23.5 mm to (173.3, 98.3), turned to 18 degrees
- moved R6 23.5 mm to (168.5, 143.3), turned to -30 degrees
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Routing:
- net Net-(U1-~{E}): track 0.00 -> 43.1 mm
- net /M1_S3: track 0.00 -> 41.7 mm
- net /M1_S2: track 0.00 -> 41.0 mm
- net /M1_S1: track 0.00 -> 29.9 mm
- net /M1: track 0.00 -> 24.0 mm
- net /M1_S0: track 0.00 -> 22.9 mm
- net Net-(D16-K): track 0.00 -> 14.1 mm
- net +3V3: track 3.81 -> 10.8 mm, vias 0 -> 1
- net Net-(U2-BOOT): track 0.00 -> 3.06 mm
- net (no net): vias 1 -> 0
Other:
- board outline removed
